File: hardware/electroNIX-USB/kicad/mcu.kicad_sch (KiCad schematic)
At the start: 27 parts, among them Q1 MMBT3904, Q2 MMBT3904, Q3 BC847, SW1 RESET, SW2 BOOT, SW3 SET, U4 ESP32-WROOM-32E-N4, U5 DS3231M

Commit message: electroNIX-USB: drop buzzer and DS3231, run stock firmware
Both builds now match a stock firmware profile with no changes:
BOARD_ELECTRONIX_3 for 4 tubes, BOARD_ELECTRONIX_4_6T for 6 tubes. Time
comes from NTP. IO0 gets a plain 10k pull-up. On the 4-tube build IO12
and IO15 are left open and reserved for anodes 5/6.

Co-Authored-By: Claude Opus 5.5 <noreply@anthropic.com>
Claude-Session: https://claude.ai/code/session_01AFMfevKEKDGbci8uJGhf4W
Parts:
- removed BT1: CR2032, Battery:BatteryHolder_Keystone_3034_1x20mm, symbol Device:Battery_Cell
- removed C11: 100n, Capacitor_SMD:C_0805_2012Metric, symbol Device:C
- removed D3: BPW34 / HPDB3J, OptoDevice:Osram_DIL2_4.3x4.65mm_P5.08mm, symbol Device:D_Photo
- removed LS1: 5 V magnetic, Buzzer_Beeper:Buzzer_12x9.5RM7.6, symbol Device:Buzzer
- removed Q3: BC847, Package_TO_SOT_SMD:SOT-23, symbol Transistor_BJT:BC847
- removed R10: 1M, Resistor_SMD:R_0805_2012Metric, symbol Device:R
- removed R11: 10k, Resistor_SMD:R_0805_2012Metric, symbol Device:R
- removed R9: 100k, Resistor_SMD:R_0805_2012Metric, symbol Device:R
- removed U5: DS3231M, Package_SO:SOIC-16W_7.5x10.3mm_P1.27mm, symbol Timer_RTC:DS3231M
- D2: value 1N4148W -> BPW34 / HPDB3J; footprint Diode_SMD:D_SOD-123 -> OptoDevice:Osram_DIL2_4.3x4.65mm_P5.08mm; symbol Device:D -> Device:D_Photo
- R6: value 4k7 -> 10k
- R7: value 4k7 -> 1M
- R8: value 1k -> 10k
Connections:
- net +5V is gone; now on net JASNOSC: D2.1 (K)
- net BUZ_N is gone; now on net GND: D2.2 (A)
- net +3V3: now also R8.1; no longer C9.1
- net BTN: now also C10.1, R8.2
- net JASNOSC: now also C9.1, R7.2; no longer C10.1
- net IO0_SCL renamed IO0
- net IO0: now also R6.2; no longer R7.2
- net IO15_SDA: no longer names the net of U4.23 (IO15)
- net IO15_SDA: no longer R6.2
- net MEL: no longer names the net of U4.14 (IO12)
- net MEL: no longer R8.1
- no-connect marks 11 -> 10
Other:
- note added: "ESP32 module (GPIO map = stock firmware BOARD_ELECTRONIX_3)"
- note added: "No buzzer and no RTC: time comes from NTP (firmware BOARD_HAS_RTC 0). IO0 has a 10k pull-up so it boots normally."
- note added: "Strapping pins at reset: IO0 high = run (10k pull-up; BOOT / auto-reset pull it low). Firmware drives IO0 as its (unfitted) buzzer pin after boot - harmless. IO2 low/float (boost gate pull-down on HV sheet) IO12 / IO15 open: internal pull-down / pull-up give the right defaults. Reserved for anodes W_5 / W_6 on the 6-tube build. IO5 SEC_1 neon driver base - default state is harmless"
- note removed: "DS3231M: optional (DNP for NTP-only builds). I2C on IO15 (SDA) / IO0 (SCL)."
- note removed: "ESP32 module (GPIO map = firmware BOARD_ELECTRONIX_3, except MEL/RTC)"
- note removed: "Strapping pins at reset: IO0 high = run (4k7 SCL pull-up; BOOT / auto-reset pull it low) IO2 low/float (boost gate pull-down on HV sheet) IO12 low = 3.3 V flash (100k pull-down on MEL) IO15 high (4k7 SDA pull-up) IO5 SEC_1 neon driver base - default state is harmless"
- moved on the sheet: C10, C9, R6, R7, R8

Commit message: electroNIX-USB: socket-adapter footprint, 0.1in neons, 4-tube PCB placement (WIP)
- Z573M socket pins on the electroNIX-2 adapter's 12.6 mm outer ring
  (default footprint), and the direct 9.53 mm footprint resized for the
  1.48 mm socket pins
- Neon_P2.54mm footprint. 6 tubes: HH:MM colon on SEC_0, MM:SS on SEC_1
- SET is a right-angle tact switch; RESET/BOOT use KMR2; low-voltage anode
  resistors moved to 0805
- source/pcb.py: builds the board from the netlist (placement, net
  classes, ESP32 antenna keepout, Freerouting, GND pours, DRC);
  source/fab.sh: fab outputs
- 4-tube board placed (102 x 66 mm, the original kit size), not yet routed

Co-Authored-By: Claude Opus 5.5 <noreply@anthropic.com>
Claude-Session: https://claude.ai/code/session_01AFMfevKEKDGbci8uJGhf4W
Parts:
- SW1, SW2: footprint Button_Switch_SMD:SW_SPST_PTS645 -> Button_Switch_SMD:SW_Push_1P1T_NO_CK_KMR2
- SW3: footprint Button_Switch_THT:SW_PUSH_6mm -> Button_Switch_THT:SW_Tactile_SPST_Angled_PTS645Vx31-2LFS
Changed lines of the file:
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@@
         (font
           (size 1.27 1.27))))
-    (property "Footprint" "Button_Switch_SMD:SW_SPST_PTS645"
+    (property "Footprint" "Button_Switch_SMD:SW_Push_1P1T_NO_CK_KMR2"
       (at 261.62 44.45 0)
       (effects
@@
         (font
           (size 1.27 1.27))))
-    (property "Footprint" "Button_Switch_SMD:SW_SPST_PTS645"
+    (property "Footprint" "Button_Switch_SMD:SW_Push_1P1T_NO_CK_KMR2"
       (at 261.62 64.77 0)
       (effects
@@
           (size 1.27 1.27))
         (justify left)))
-    (property "Footprint" "Button_Switch_THT:SW_PUSH_6mm"
+    (property "Footprint" "Button_Switch_THT:SW_Tactile_SPST_Angled_PTS645Vx31-2LFS"
       (at 384.81 160.02 90)
       (effects

Commit message: electroNIX-USB: drop all switches, regroup board placement by circuit
- No RESET/BOOT/SET: the firmware reads no button, and the CH340C
  DTR/RTS auto-reset handles flashing. SET's pull-up and cap are gone.
- Boost converter is a compact loop (input caps -> L1 -> FET tab) feeding
  the multiplier columns in chain order.
- ESP32: 3V3 decoupling at pin 2, EN RC at pin 3, HV feedback divider and
  clamp at IO35; auto-reset between the CH340C and the module's UART pins.
- Front band spread out: output cap + KBIAS left, cathode row, one anode
  cluster under each tube.
- 6-tube board placed too (150 x 66 mm). Both boards unrouted.

Co-Authored-By: Claude Opus 5.5 <noreply@anthropic.com>
Claude-Session: https://claude.ai/code/session_01AFMfevKEKDGbci8uJGhf4W
Parts:
- removed C10: 100n, Capacitor_SMD:C_0805_2012Metric, symbol Device:C
- removed R8: 10k, Resistor_SMD:R_0805_2012Metric, symbol Device:R
- removed SW1: RESET, Button_Switch_SMD:SW_Push_1P1T_NO_CK_KMR2, symbol Switch:SW_Push
- removed SW2: BOOT, Button_Switch_SMD:SW_Push_1P1T_NO_CK_KMR2, symbol Switch:SW_Push
- removed SW3: SET, Button_Switch_THT:SW_Tactile_SPST_Angled_PTS645Vx31-2LFS, symbol Switch:SW_Push
Connections:
- net BTN: no longer names the net of U4.4 (SENSOR_VP)
- no-connect marks 10 -> 11
Other:
- note added: "No buttons: the CH340C resets the ESP32 and enters download mode through DTR/RTS; unplugging USB is the reset. Recovery if auto-reset ever fails: short the IO0 pull-up (the 10k on IO0) to GND while plugging in."
- note added: "Reset and auto-program (DTR/RTS) - no RESET/BOOT buttons needed"
- note removed: "Reset, boot and auto-program (DTR/RTS)"
