File: hardware/electroNIX-USB/kicad/display.kicad_sch (KiCad schematic)
At the start: 69 parts, among them Q10 MMBTA92, Q11 MMBTA42, Q12 MMBTA92, Q13 MMBTA42, Q14 MMBTA42, Q15 MMBTA42, Q16 MMBTA42, Q17 MMBTA42, Q18 MMBTA42, Q19 MMBTA42, Q20 MMBTA42, Q21 MMBTA42, Q22 MMBTA42, Q23 MMBTA42, Q24 MMBTA42, Q5 MMBTA42, Q6 MMBTA92, Q7 MMBTA42, Q8 MMBTA92, Q9 MMBTA42

Commit message: electroNIX-USB: add 6-tube variant
The generator takes --tubes 4|6. The 6-tube build adds two anode switches
on IO12/IO15 and doubles the colon neons. It drops the buzzer and DS3231,
which matches the stock BOARD_ELECTRONIX_4_6T GPIO map, so no firmware
change is needed. HV supply, cathode drivers, ESP32, USB and power are
unchanged. Both projects are committed, with their own schematic PDF
and BOM.

Co-Authored-By: Claude Opus 5.5 <noreply@anthropic.com>
Claude-Session: https://claude.ai/code/session_01AFMfevKEKDGbci8uJGhf4W
Parts:
- R42, R44: value 100k -> 47k
Connections:
- net NEK_1: now reaches NE2.1, Q24.3 (C)
- net NEK_0: now reaches NE1.1, Q23.3 (C)
Other:
- note added: "Original Z573M kit fits one neon (SEC_0). Fit the second for a two-dot colon; Firmware drives SEC_0/SEC_1 independently. 150k per neon: ~0.6 mA at 170 V."
- note added: "W_n high -> tube n anode at +170V through 10k. Anode current ~2 mA peak. 6-tube build (--tubes 6): two more of these on IO12/IO15."
- note removed: "Original Z573M kit fits one neon (SEC_0). Fit the second for a two-dot colon; firmware drives them independently. 150k: ~0.6 mA at 170 V."
- note removed: "W_n high -> tube n anode at +170V through 10k. Anode current ~2 mA peak."
- moved on the sheet: NE2, Q23, R42, R45
Changed lines of the file:
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@@
   (wire
     (pts
-      (xy 436.88 110.49)
-      (xy 434.34 110.49))
+      (xy 426.72 110.49)
+      (xy 424.18 110.49))
     (stroke
       (width 0)
@@
   (wire
     (pts
-      (xy 452.12 115.57)
-      (xy 452.12 118.11))
+      (xy 441.96 115.57)
+      (xy 441.96 118.11))
+    (stroke
+      (width 0)
+      (type default))
+)
+  (wire
+    (pts
+      (xy 441.96 105.41)
+      (xy 441.96 102.87))
+    (stroke
+      (width 0)
+      (type default))
+)
+  (wire
+    (pts
+      (xy 452.12 105.41)
+      (xy 452.12 107.95))
     (stroke
       (width 0)
@@
   (wire
     (pts
-      (xy 513.08 87.63)
-      (xy 513.08 85.09))
+      (xy 513.08 105.41)
+      (xy 513.08 102.87))
+    (stroke
+      (width 0)
+      (type default))
+)
+  (wire
+    (pts
+      (xy 523.24 105.41)
+      (xy 523.24 107.95))
+    (stroke
+      (width 0)
+      (type default))
+)
+  (wire
+    (pts
+      (xy 523.24 87.63)
+      (xy 523.24 85.09))
     (stroke
       (width 0)
@@
   (global_label "SEC_0"
     (shape passive)
-    (at 434.34 110.49 180)
+    (at 424.18 110.49 180)
     (fields_autoplaced)
     (effects
@@
       (justify right))
     (property "Intersheetrefs" "${INTERSHEET_REFS}"
-      (at 434.34 110.49 0)
+      (at 424.18 110.49 0)
       (effects
         (font
           (size 1.27 1.27)) hide)))
+  (label "NEK_0"
+    (at 441.96 102.87 90)
+    (fields_autoplaced)
+    (effects
+      (font
+        (size 1.27 1.27))
+      (justify left bottom))
+)
+  (label "NEK_0"
+    (at 452.12 107.95 270)
+    (fields_autoplaced)
+    (effects
+      (font
+        (size 1.27 1.27))
+      (justify right bottom))
+)
   (global_label "SEC_1"
     (shape passive)
@@
         (font
           (size 1.27 1.27)) hide)))
+  (label "NEK_1"
+    (at 513.08 102.87 90)
+    (fields_autoplaced)
+    (effects
+      (font
+        (size 1.27 1.27))
+      (justify left bottom))
+)
+  (label "NEK_1"
+    (at 523.24 107.95 270)
+    (fields_autoplaced)
+    (effects
+      (font
+        (size 1.27 1.27))
+      (justify right bottom))
+)
   (label "K_0"
     (at 425.45 193.04 90)
@@
       (justify left top))
 )
-  (text "W_n high -> tube n anode at +170V through 10k. Anode current ~2 mA peak."
+  (text "W_n high -> tube n anode at +170V through 10k. Anode current ~2 mA peak.  6-tube build (--tubes 6): two more of these on IO12/IO15."
     (at 25 98 0)
     (effects
@@
       (justify left top))
 )
-  (text "Original Z573M kit fits one neon (SEC_0). Fit the second for a two-dot colon;\nfirmware drives them independently. 150k: ~0.6 mA at 170 V."
+  (text "Original Z573M kit fits one neon (SEC_0). Fit the second for a two-dot colon;\nFirmware drives SEC_0/SEC_1 independently. 150k per neon: ~0.6 mA at 170 V."
     (at 415 125 0)
     (effects
@@
     (dnp no)
     (property "Reference" "N1"
-      (at 44 151 0)
+      (at 43.69 151 0)
       (effects
         (font
@@
         (justify left)))
     (property "Value" "Z573M"
-      (at 64 151 0)
+      (at 63.69 151 0)
       (effects
         (font
@@
     (dnp no)
     (property "Reference" "N2"
-      (at 134 151 0)
+      (at 133.86 151 0)
       (effects
         (font
@@
         (justify left)))
     (property "Value" "Z573M"
-      (at 154 151 0)
+      (at 153.86 151 0)
       (effects
         (font
@@
     (dnp no)
     (property "Reference" "N3"
-      (at 224 151 0)
+      (at 224.03 151 0)
       (effects
         (font
@@
         (justify left)))
     (property "Value" "Z573M"
-      (at 244 151 0)
+      (at 244.03 151 0)
       (effects
         (font
@@
     (dnp no)
     (property "Reference" "N4"
-      (at 314 151 0)
+      (at 314.2 151 0)
       (effects
         (font
@@
         (justify left)))
     (property "Value" "Z573M"
-      (at 334 151 0)
+      (at 334.2 151 0)
       (effects
         (font
@@
   (symbol
     (lib_id "Device:R")
-    (at 440.69 110.49 90)
+    (at 430.53 110.49 90)
     (unit 1)
     (in_bom yes)
@@
     (dnp no)
     (property "Reference" "R42"
-      (at 440.69 107.95 90)
+      (at 430.53 107.95 90)
       (effects
         (font
           (size 1.27 1.27))))
-    (property "Value" "100k"
-      (at 440.69 113.03 90)
+    (property "Value" "47k"
+      (at 430.53 113.03 90)
       (effects
         (font
           (size 1.27 1.27))))
     (property "Footprint" "Resistor_SMD:R_0805_2012Metric"
-      (at 440.69 110.49 90)
+      (at 430.53 110.49 90)
       (effects
         (font
@@
         (justify left) hide))
     (property "Datasheet" "~"
-      (at 440.69 110.49 90)
+      (at 430.53 110.49 90)
       (effects
         (font
@@
   (symbol
     (lib_id "power:GND")
-    (at 452.12 118.11 0)
+    (at 441.96 118.11 0)
     (unit 1)
     (in_bom yes)
@@
     (dnp no)
     (property "Reference" "#PWR5071"
-      (at 452.12 118.11 0)
+      (at 441.96 118.11 0)
       (effects
         (font
           (size 1.27 1.27)) hide))
     (property "Value" "GND"
-      (at 452.12 121.31 0)
+      (at 441.96 121.31 0)
       (effects
         (font
           (size 1.27 1.27))))
     (property "Footprint" ""
-      (at 452.12 118.11 0)
+      (at 441.96 118.11 0)
       (effects
         (font
           (size 1.27 1.27)) hide))
     (property "Datasheet" ""
-      (at 452.12 118.11 0)
+      (at 441.96 118.11 0)
       (effects
         (font
@@
   (symbol
     (lib_id "Transistor_BJT:MMBTA42")
-    (at 449.58 110.49 0)
+    (at 439.42 110.49 0)
     (unit 1)
     (in_bom yes)
@@
     (dnp no)
     (property "Reference" "Q23"
-      (at 453.39 109.22 0)
+      (at 443.23 109.22 0)
       (effects
         (font
@@
         (justify left)))
     (property "Value" "MMBTA42"
-      (at 453.39 111.76 0)
+      (at 443.23 111.76 0)
       (effects
         (font
@@
         (justify left)))
     (property "Footprint" "Package_TO_SOT_SMD:SOT-23"
-      (at 449.58 110.49 0)
+      (at 439.42 110.49 0)
       (effects
         (font
@@
         (justify left) hide))
     (property "Datasheet" "~"
-      (at 449.58 110.49 0)
+      (at 439.42 110.49 0)
       (effects
         (font
@@
         (font
           (size 1.27 1.27))))
-    (property "Value" "100k"
+    (property "Value" "47k"
       (at 501.65 113.03 90)
       (effects
@@
   (symbol
     (lib_id "Device:Lamp_Neon")
-    (at 513.08 100.33 0)
+    (at 523.24 100.33 0)
     (unit 1)
     (in_bom yes)
@@
     (dnp no)
     (property "Reference" "NE2"
-      (at 514.35 99.06 0)
+      (at 524.51 99.06 0)
       (effects
         (font
@@
         (justify left)))
     (property "Value" "NE-2 / INS-1"
-      (at 514.35 101.6 0)
+      (at 524.51 101.6 0)
       (effects
         (font
@@
         (justify left)))
     (property "Footprint" ""
-      (at 513.08 100.33 0)
+      (at 523.24 100.33 0)
       (effects
         (font
@@
         (justify left) hide))
     (property "Datasheet" "~"
-      (at 513.08 100.33 0)
+      (at 523.24 100.33 0)
       (effects
         (font
@@
   (symbol
     (lib_id "electronix:+170V")
-    (at 513.08 85.09 0)
+    (at 523.24 85.09 0)
     (unit 1)
     (in_bom yes)
@@
     (dnp no)
     (property "Reference" "#PWR5080"
-      (at 513.08 85.09 0)
+      (at 523.24 85.09 0)
       (effects
         (font
           (size 1.27 1.27)) hide))
     (property "Value" "+170V"
-      (at 513.08 81.89 0)
+      (at 523.24 81.89 0)
       (effects
         (font
           (size 1.27 1.27))))
     (property "Footprint" ""
-      (at 513.08 85.09 0)
+      (at 523.24 85.09 0)
       (effects
         (font
           (size 1.27 1.27)) hide))
     (property "Datasheet" ""
-      (at 513.08 85.09 0)
+      (at 523.24 85.09 0)
       (effects
         (font
@@
   (symbol
     (lib_id "Device:R")
-    (at 513.08 91.44 0)
+    (at 523.24 91.44 0)
     (unit 1)
     (in_bom yes)
@@
     (dnp no)
     (property "Reference" "R45"
-      (at 514.35 90.17 0)
+      (at 524.51 90.17 0)
       (effects
         (font
@@
         (justify left)))
     (property "Value" "150k"
-      (at 514.35 92.71 0)
+      (at 524.51 92.71 0)
       (effects
         (font
@@
         (justify left)))
     (property "Footprint" "Resistor_SMD:R_1206_3216Metric"
-      (at 513.08 91.44 0)
+      (at 523.24 91.44 0)
       (effects
         (font
@@
         (justify left) hide))
     (property "Datasheet" "~"
-      (at 513.08 91.44 0)
+      (at 523.24 91.44 0)
       (effects
         (font

Commit message: electroNIX-USB: drop buzzer and DS3231, run stock firmware
Both builds now match a stock firmware profile with no changes:
BOARD_ELECTRONIX_3 for 4 tubes, BOARD_ELECTRONIX_4_6T for 6 tubes. Time
comes from NTP. IO0 gets a plain 10k pull-up. On the 4-tube build IO12
and IO15 are left open and reserved for anodes 5/6.

Co-Authored-By: Claude Opus 5.5 <noreply@anthropic.com>
Claude-Session: https://claude.ai/code/session_01AFMfevKEKDGbci8uJGhf4W
Parts:
- removed C23: 2u2 50V, Capacitor_SMD:C_1206_3216Metric, symbol Device:C
- removed D21: 1N4148W, Diode_SMD:D_SOD-123, symbol Device:D
- removed Q24: MMBTA42, Package_TO_SOT_SMD:SOT-23, symbol Transistor_BJT:MMBTA42
- removed R45: 150k, Resistor_SMD:R_1206_3216Metric, symbol Device:R
- removed R46: 430k, Resistor_SMD:R_1206_3216Metric, symbol Device:R
- removed R47: 100k, Resistor_SMD:R_0805_2012Metric, symbol Device:R
- added C22: 2u2 50V, Capacitor_SMD:C_1206_3216Metric, symbol Device:C
- added D11: 1N4148W, Diode_SMD:D_SOD-123, symbol Device:D
- added Q4: MMBTA42, Package_TO_SOT_SMD:SOT-23, symbol Transistor_BJT:MMBTA42
- added R13: 15k, Resistor_SMD:R_0805_2012Metric, symbol Device:R
- added R14: 430k, Resistor_SMD:R_1206_3216Metric, symbol Device:R
- added R15: 100k, Resistor_SMD:R_1206_3216Metric, symbol Device:R
- Q10, Q12, Q6, Q8: value MMBTA92 -> MMBTA42; symbol Transistor_BJT:MMBTA92 -> Transistor_BJT:MMBTA42
- Q11, Q5, Q7, Q9: value MMBTA42 -> MMBTA92; symbol Transistor_BJT:MMBTA42 -> Transistor_BJT:MMBTA92
- R16, R20, R24, R28: value 15k -> 10k; footprint Resistor_SMD:R_0805_2012Metric -> Resistor_SMD:R_1206_3216Metric
- R17, R21, R25, R29: value 430k -> 15k; footprint Resistor_SMD:R_1206_3216Metric -> Resistor_SMD:R_0805_2012Metric
- R18, R22, R26: value 100k -> 430k
- R19, R23, R27: value 10k -> 100k
- R30: value 100k -> 15k; footprint Resistor_SMD:R_1206_3216Metric -> Resistor_SMD:R_0805_2012Metric
- R31: value 10k -> 15k; footprint Resistor_SMD:R_1206_3216Metric -> Resistor_SMD:R_0805_2012Metric
- R39, R41: value 15k -> 47k
- R40: value 15k -> 150k; footprint Resistor_SMD:R_0805_2012Metric -> Resistor_SMD:R_1206_3216Metric
- R42: value 47k -> 150k; footprint Resistor_SMD:R_0805_2012Metric -> Resistor_SMD:R_1206_3216Metric
- R43: value 150k -> 430k
- R44: value 47k -> 100k
Connections:
- net +170V: now also Q11.2 (E), Q5.2 (E), Q7.2 (E), Q9.2 (E), R19.1, R23.1, R27.1, R40.1, R42.1, R15.1; no longer Q10.2 (E), Q12.2 (E), Q6.2 (E), Q8.2 (E), R18.1, R22.1, R26.1, R30.1
- net A_1: now also R16.2; no longer R19.2
- net A_2: now also R20.2; no longer R23.2
- net A_3: now also R24.2; no longer R27.2
- net A_4: now also R28.2; no longer R31.2
- net C_0: now also R29.1; no longer R32.1
- net C_1: now also R30.1; no longer R33.1
- net C_2: now also R31.1; no longer R34.1
- net C_3: now also R32.1; no longer R35.1
- net C_4: now also R33.1; no longer R36.1
- net C_5: now also R34.1; no longer R37.1
- net C_6: now also R35.1; no longer R38.1
- net C_7: now also R36.1; no longer R39.1
- net C_8: now also R37.1; no longer R40.1
- net C_9: now also R38.1; no longer R41.1
- net GND: now also Q10.2 (E), Q12.2 (E), Q6.2 (E), Q8.2 (E), R44.2, C22.2, Q4.2 (E); no longer Q11.2 (E), Q5.2 (E), Q7.2 (E), Q9.2 (E)
- net KBIAS: now also R43.2, R44.1, C22.1, D11.1 (K)
- net K_0: now also Q12.3 (C), D11.2 (A); no longer D12.2 (A), Q13.3 (C)
- net K_1: now also D12.2 (A), Q13.3 (C); no longer D13.2 (A), Q14.3 (C)
- net K_2: now also D13.2 (A), Q14.3 (C); no longer D14.2 (A), Q15.3 (C)
- net K_3: now also D14.2 (A), Q15.3 (C); no longer D15.2 (A), Q16.3 (C)
- net K_4: now also D15.2 (A), Q16.3 (C); no longer D16.2 (A), Q17.3 (C)
- net K_5: now also D16.2 (A), Q17.3 (C); no longer D17.2 (A), Q18.3 (C)
- net K_6: now also D17.2 (A), Q18.3 (C); no longer D18.2 (A), Q19.3 (C)
- net K_7: now also D18.2 (A), Q19.3 (C); no longer D19.2 (A), Q20.3 (C)
- net K_8: now also D19.2 (A), Q20.3 (C); no longer D20.2 (A), Q21.3 (C)
- net K_9: now also D20.2 (A), Q21.3 (C); no longer Q22.3 (C)
- net NEK_0: now also Q22.3 (C); no longer Q23.3 (C)
- net NEK_1: now also Q23.3 (C)
- net SEC_0: now also R39.1; no longer R42.1
- net SEC_1: now also R41.1; no longer R44.1
- net W_1: now also R13.1; no longer R16.1
- net W_2: now also R17.1; no longer R20.1
- net W_3: now also R21.1; no longer R24.1
- net W_4: now also R25.1; no longer R28.1
- net at Q6.3 (C): now also R18.2; no longer R19.1
- net at Q7.1 (B): now also R18.1, R19.2; no longer R20.2
- net at Q9.1 (B): now also R22.1, R23.2; no longer R24.2
- net at Q11.1 (B): now also R26.1, R27.2; no longer R28.2
- net at Q5.1 (B): now also R14.1, R15.2; no longer R16.2
- net at R17.2: now also Q6.1 (B); no longer Q5.3 (C)
- net at Q20.1 (B): now also R37.2; no longer R39.2
- net at R34.2: now also Q17.1 (B); no longer Q15.1 (B)
- net at Q14.1 (B): now also R31.2; no longer R33.2
- net at R36.2: now also Q19.1 (B); no longer Q17.1 (B)
- net at Q11.3 (C): now also R28.1; no longer R29.2
- net at R40.2: now also NE1.2; no longer Q21.1 (B)
- net at Q7.3 (C): now also R20.1; no longer R21.2
- net at Q18.1 (B): now also R35.2; no longer R37.2
- net at Q8.3 (C): now also R22.2; no longer R23.1
- net at NE2.2: now also R42.2
- net at Q10.3 (C): now also R26.2; no longer R27.1
- net at Q13.1 (B): now also R30.2; no longer R32.2
- net at R41.2: now also Q23.1 (B); no longer Q22.1 (B)
- net at Q9.3 (C): now also R24.1; no longer R25.2
- net at R38.2: now also Q21.1 (B); no longer Q19.1 (B)
- net at Q16.1 (B): now also R33.2; no longer R35.2
- new net: Q5.3 (C), R16.1
- new net: Q12.1 (B), R29.2
- new net: Q4.1 (B), R13.2
- new net: Q4.3 (C), R14.2
- new net: Q8.1 (B), R21.2
- new net: Q10.1 (B), R25.2
- new net: Q15.1 (B), R32.2
- new net: Q22.1 (B), R39.2
Other:
- moved on the sheet: D12, D13, D14, D15, D16, D17, D18, D19, D20, Q13, Q14, Q15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

Commit message: electroNIX-USB: apply RFT Z573M data sheet, add tube footprint
The data book confirms the pinout already in the symbol. The tube is
side-view (not top-view), with 13 flying leads on a 9.53 mm circle and
wire 7 at the front. New footprint electronix:Nixie_RFT_Z573M (top
view, wire 7 toward the front edge) is assigned to the tubes.

Tube current: Ik is 1.5-2.5 mA continuous, 12 mA pulse. PCB-036's 10k
anode resistors averaged only ~0.75 mA per tube when multiplexed. Anode
resistors are now 5k6 (4 tubes) and 3k9 (6 tubes), cathode base
resistors 6k8. To carry the extra HV power, the ladder caps go to
2.2 uF and the 6-tube build uses a 22 uH inductor.

Co-Authored-By: Claude Opus 5.5 <noreply@anthropic.com>
Claude-Session: https://claude.ai/code/session_01AFMfevKEKDGbci8uJGhf4W
Parts:
- N1, N2, N3, N4: footprint (none) -> electronix:Nixie_RFT_Z573M
- R16, R20, R24, R28: value 10k -> 5k6
- R29, R30, R31, R32, R33, R34, R35, R36, R37, R38: value 15k -> 6k8
Other:
- note added: "Pin 4 = internal connection (leave open). Pin 10 = decimal point (unused). Pinout per RFT data book (frank.pocnet.net/sheets/084/z/Z573M.pdf)."
- note added: "Tubes (RFT Z573M side-view, 13 flying leads on 9.53 mm circle, wire 7 at front)"
- note added: "W_n high -> tube n anode at +170V through 5k6: ~5.4 mA peak at 170 V, ~1.3 mA average per tube (Z573M: 1.5-2.5 mA cont., 12 mA pulse). Peak current follows (V_HV - 140 V): keep the firmware HV setpoint <= 180 V. 6-tube build (--tubes 6): two more of these on IO12/IO15."
- note removed: "Pin 4 = internal connection (leave open). Pin 10 = PR sign (unused). Pinout from tube-tester.com Z573M page; check against a real tube before layout."
- note removed: "Tubes (RFT Z573M, B13D base, pin 7 at front)"
- note removed: "W_n high -> tube n anode at +170V through 10k. Anode current ~2 mA peak. 6-tube build (--tubes 6): two more of these on IO12/IO15."
Changed lines of the file:
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@@
       (justify left top))
 )
-  (text "W_n high -> tube n anode at +170V through 10k. Anode current ~2 mA peak.  6-tube build (--tubes 6): two more of these on IO12/IO15."
-    (at 25 98 0)
+  (text "W_n high -> tube n anode at +170V through 5k6: ~5.4 mA peak at 170 V, ~1.3 mA average per tube (Z573M: 1.5-2.5 mA cont., 12 mA pulse).\nPeak current follows (V_HV - 140 V): keep the firmware HV setpoint <= 180 V.  6-tube build (--tubes 6): two more of these on IO12/IO15."
+    (at 25 95 0)
     (effects
       (font
@@
       (type none))
 )
-  (text "Tubes (RFT Z573M, B13D base, pin 7 at front)"
+  (text "Tubes (RFT Z573M side-view, 13 flying leads on 9.53 mm circle, wire 7 at front)"
     (at 21.27 116.27 0)
     (effects
@@
       (justify left top))
 )
-  (text "Pin 4 = internal connection (leave open). Pin 10 = PR sign (unused).\nPinout from tube-tester.com Z573M page; check against a real tube before layout."
+  (text "Pin 4 = internal connection (leave open). Pin 10 = decimal point (unused).\nPinout per RFT data book (frank.pocnet.net/sheets/084/z/Z573M.pdf)."
     (at 25 195 0)
     (effects
@@
           (size 1.27 1.27))
         (justify left)))
-    (property "Value" "10k"
+    (property "Value" "5k6"
       (at 60.96 77.47 0)
       (effects
@@
           (size 1.27 1.27))
         (justify left)))
-    (property "Value" "10k"
+    (property "Value" "5k6"
       (at 151.13 77.47 0)
       (effects
@@
           (size 1.27 1.27))
         (justify left)))
-    (property "Value" "10k"
+    (property "Value" "5k6"
       (at 241.3 77.47 0)
       (effects
@@
           (size 1.27 1.27))
         (justify left)))
-    (property "Value" "10k"
+    (property "Value" "5k6"
       (at 331.47 77.47 0)
       (effects
@@
           (size 1.27 1.27))
         (justify left)))
-    (property "Footprint" ""
+    (property "Footprint" "electronix:Nixie_RFT_Z573M"
       (at 59.69 160.02 0)
       (effects
@@
           (size 1.27 1.27))
         (justify left)))
-    (property "Footprint" ""
+    (property "Footprint" "electronix:Nixie_RFT_Z573M"
       (at 149.86 160.02 0)
       (effects
@@
           (size 1.27 1.27))
         (justify left)))
-    (property "Footprint" ""
+    (property "Footprint" "electronix:Nixie_RFT_Z573M"
       (at 240.03 160.02 0)
       (effects
@@
           (size 1.27 1.27))
         (justify left)))
-    (property "Footprint" ""
+    (property "Footprint" "electronix:Nixie_RFT_Z573M"
       (at 330.2 160.02 0)
       (effects
@@
         (font
           (size 1.27 1.27))))
-    (property "Value" "15k"
+    (property "Value" "6k8"
       (at 35.56 273.05 90)
       (effects
@@
         (font
           (size 1.27 1.27))))
-    (property "Value" "15k"
+    (property "Value" "6k8"
       (at 72.39 273.05 90)
       (effects
@@
         (font
           (size 1.27 1.27))))
-    (property "Value" "15k"
+    (property "Value" "6k8"
       (at 107.95 273.05 90)
       (effects
@@
         (font
           (size 1.27 1.27))))
-    (property "Value" "15k"
+    (property "Value" "6k8"
       (at 143.51 273.05 90)
       (effects
@@
         (font
           (size 1.27 1.27))))
-    (property "Value" "15k"
+    (property "Value" "6k8"
       (at 180.34 273.05 90)
       (effects
@@
         (font
           (size 1.27 1.27))))
-    (property "Value" "15k"
+    (property "Value" "6k8"
       (at 215.9 273.05 90)
       (effects
@@
         (font
           (size 1.27 1.27))))
-    (property "Value" "15k"
+    (property "Value" "6k8"
       (at 252.73 273.05 90)
       (effects
@@
         (font
           (size 1.27 1.27))))
-    (property "Value" "15k"
+    (property "Value" "6k8"
       (at 288.29 273.05 90)
       (effects
@@
         (font
           (size 1.27 1.27))))
-    (property "Value" "15k"
+    (property "Value" "6k8"
       (at 323.85 273.05 90)
       (effects
@@
         (font
           (size 1.27 1.27))))
-    (property "Value" "15k"
+    (property "Value" "6k8"
       (at 360.68 273.05 90)
       (effects
