File: hardware/electroNIX-USB/kicad/hv_supply.kicad_sch (KiCad schematic)
At the start: 25 parts, among them Q4 IRLR3110ZPBF

Commit message: electroNIX-USB: drop buzzer and DS3231, run stock firmware
Both builds now match a stock firmware profile with no changes:
BOARD_ELECTRONIX_3 for 4 tubes, BOARD_ELECTRONIX_4_6T for 6 tubes. Time
comes from NTP. IO0 gets a plain 10k pull-up. On the 4-tube build IO12
and IO15 are left open and reserved for anodes 5/6.

Co-Authored-By: Claude Opus 5.5 <noreply@anthropic.com>
Claude-Session: https://claude.ai/code/session_01AFMfevKEKDGbci8uJGhf4W
Parts:
- removed C22: 100n, Capacitor_SMD:C_0805_2012Metric, symbol Device:C
- removed D11: BAT54S, Package_TO_SOT_SMD:SOT-23, symbol Diode:BAT54S
- removed Q4: IRLR3110ZPBF, Package_TO_SOT_SMD:TO-252-2, symbol Device:Q_NMOS_GDS
- removed R13: 10k, Resistor_SMD:R_0805_2012Metric, symbol Device:R
- removed R14: 430k, Resistor_SMD:R_1206_3216Metric, symbol Device:R
- removed R15: 6k2, Resistor_SMD:R_0805_2012Metric, symbol Device:R
- added C11: 22u 10V, Capacitor_SMD:C_1206_3216Metric, symbol Device:C
- added D3: 10MQ100N, Diode_SMD:D_SMA, symbol Device:D_Schottky
- added Q3: IRLR3110ZPBF, Package_TO_SOT_SMD:TO-252-2, symbol Device:Q_NMOS_GDS
- added R10: 10k, Resistor_SMD:R_0805_2012Metric, symbol Device:R
- added R11: 430k, Resistor_SMD:R_1206_3216Metric, symbol Device:R
- added R9: 10R, Resistor_SMD:R_0805_2012Metric, symbol Device:R
- C12: value 22u 10V -> 100n; footprint Capacitor_SMD:C_1206_3216Metric -> Capacitor_SMD:C_0805_2012Metric
- C13: value 100n -> 1u 100V; footprint Capacitor_SMD:C_0805_2012Metric -> Capacitor_SMD:C_1210_3225Metric
- C20: value 1u 100V -> 2u2 250V; footprint Capacitor_SMD:C_1210_3225Metric -> Capacitor_THT:CP_Radial_D6.3mm_P2.50mm; symbol Device:C -> Device:C_Polarized
- C21: value 2u2 250V -> 100n; footprint Capacitor_THT:CP_Radial_D6.3mm_P2.50mm -> Capacitor_SMD:C_0805_2012Metric; symbol Device:C_Polarized -> Device:C
- D10: value 10MQ100N -> BAT54S; footprint Diode_SMD:D_SMA -> Package_TO_SOT_SMD:SOT-23; symbol Device:D_Schottky -> Diode:BAT54S
- R12: value 10R -> 6k2
Connections:
- net +170V: now also C13.1, C20.1, D3.1 (K), R11.1; no longer C14.1, C21.1, D4.1 (K)
- net +3V3: now also D10.2 (K)
- net +5V: now also C11.1; no longer C13.1
- net CW_B1: now also C18.2, C19.1, D7.2 (A), D8.1 (K); no longer C19.2, C20.1, D8.2 (A), D9.1 (K)
- net CW_B2: now also C17.2, C18.1, D5.2 (A), D6.1 (K); no longer C18.2, C19.1, D6.2 (A), D7.1 (K)
- net CW_B3: now also C17.1, D4.1 (K), D3.2 (A); no longer C18.1, D4.2 (A), D5.1 (K)
- net CW_T1: now also C15.2, C16.1, D8.2 (A), D9.1 (K); no longer C16.2, C17.1, D10.1 (K), D9.2 (A)
- net CW_T2: now also C14.2, C15.1, D6.2 (A), D7.1 (K); no longer C15.2, C16.1, D7.2 (A), D8.1 (K)
- net CW_T3: now also C13.2, C14.1, D4.2 (A), D5.1 (K); no longer C14.2, C15.1, D5.2 (A), D6.1 (K)
- net GND: now also C16.2, C20.2, D10.1 (A), R12.2, C11.2, Q3.3 (S), R10.2; no longer C13.2, C17.2
- net HV_SW: now also C19.2, D9.2 (A), Q3.2 (D); no longer C20.2, D10.2 (A)
- net KOMP_170V: now also C21.1, D10.3 (COM), R12.1, R11.2
- net PWM: now also R10.1, R9.1; no longer R12.1
- new net: Q3.1 (G), R9.2
Other:
- moved on the sheet: C12, C13, C14, C15, C16, C17, C18, C19, D4, D5, D6, D7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
Changed lines of the file:
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@@
     (on_board yes)
     (dnp no)
-    (property "Reference" "C12"
+    (property "Reference" "C11"
       (at 36.83 58.42 0)
       (effects
@@
       (project "electroNIX-USB"
         (path "/af167dc7-e2c9-570c-bdf4-28156a519677/f6fa350a-459e-5361-98c1-1f12d068c3cb"
-          (reference "C12")
+          (reference "C11")
           (unit 1)))))
   (symbol
@@
     (on_board yes)
     (dnp no)
-    (property "Reference" "C13"
+    (property "Reference" "C12"
       (at 48.26 58.42 0)
       (effects
@@
       (project "electroNIX-USB"
         (path "/af167dc7-e2c9-570c-bdf4-28156a519677/f6fa350a-459e-5361-98c1-1f12d068c3cb"
-          (reference "C13")
+          (reference "C12")
           (unit 1)))))
   (symbol
@@
     (on_board yes)
     (dnp no)
-    (property "Reference" "Q4"
+    (property "Reference" "Q3"
       (at 104.14 78.74 0)
       (effects
@@
       (project "electroNIX-USB"
         (path "/af167dc7-e2c9-570c-bdf4-28156a519677/f6fa350a-459e-5361-98c1-1f12d068c3cb"
-          (reference "Q4")
+          (reference "Q3")
           (unit 1)))))
   (symbol
@@
     (on_board yes)
     (dnp no)
-    (property "Reference" "R12"
+    (property "Reference" "R9"
       (at 91.44 77.47 90)
       (effects
@@
       (project "electroNIX-USB"
         (path "/af167dc7-e2c9-570c-bdf4-28156a519677/f6fa350a-459e-5361-98c1-1f12d068c3cb"
-          (reference "R12")
+          (reference "R9")
           (unit 1)))))
   (symbol
@@
     (on_board yes)
     (dnp no)
-    (property "Reference" "R13"
+    (property "Reference" "R10"
       (at 86.36 93.98 0)
       (effects
@@
       (project "electroNIX-USB"
         (path "/af167dc7-e2c9-570c-bdf4-28156a519677/f6fa350a-459e-5361-98c1-1f12d068c3cb"
-          (reference "R13")
+          (reference "R10")
           (unit 1)))))
   (symbol
@@
     (on_board yes)
     (dnp no)
-    (property "Reference" "C14"
+    (property "Reference" "C13"
       (at 199.39 46.99 90)
       (effects
@@
       (project "electroNIX-USB"
         (path "/af167dc7-e2c9-570c-bdf4-28156a519677/f6fa350a-459e-5361-98c1-1f12d068c3cb"
-          (reference "C14")
+          (reference "C13")
           (unit 1)))))
   (symbol
@@
     (on_board yes)
     (dnp no)
-    (property "Reference" "C15"
+    (property "Reference" "C14"
       (at 250.19 46.99 90)
       (effects
@@
       (project "electroNIX-USB"
         (path "/af167dc7-e2c9-570c-bdf4-28156a519677/f6fa350a-459e-5361-98c1-1f12d068c3cb"
-          (reference "C15")
+          (reference "C14")
           (unit 1)))))
   (symbol
@@
     (on_board yes)
     (dnp no)
-    (property "Reference" "C16"
+    (property "Reference" "C15"
       (at 299.72 46.99 90)
       (effects
@@
       (project "electroNIX-USB"
         (path "/af167dc7-e2c9-570c-bdf4-28156a519677/f6fa350a-459e-5361-98c1-1f12d068c3cb"
-          (reference "C16")
+          (reference "C15")
           (unit 1)))))
   (symbol
@@
     (on_board yes)
     (dnp no)
-    (property "Reference" "C17"
+    (property "Reference" "C16"
       (at 350.52 46.99 90)
       (effects
@@
       (project "electroNIX-USB"
         (path "/af167dc7-e2c9-570c-bdf4-28156a519677/f6fa350a-459e-5361-98c1-1f12d068c3cb"
-          (reference "C17")
+          (reference "C16")
           (unit 1)))))
   (symbol
@@
     (on_board yes)
     (dnp no)
-    (property "Reference" "C18"
+    (property "Reference" "C17"
       (at 224.79 92.71 90)
       (effects
@@
       (project "electroNIX-USB"
         (path "/af167dc7-e2c9-570c-bdf4-28156a519677/f6fa350a-459e-5361-98c1-1f12d068c3cb"
-          (reference "C18")
+          (reference "C17")
           (unit 1)))))
   (symbol
@@
     (on_board yes)
     (dnp no)
-    (property "Reference" "C19"
+    (property "Reference" "C18"
       (at 275.59 92.71 90)
       (effects
@@
       (project "electroNIX-USB"
         (path "/af167dc7-e2c9-570c-bdf4-28156a519677/f6fa350a-459e-5361-98c1-1f12d068c3cb"
-          (reference "C19")
+          (reference "C18")
           (unit 1)))))
   (symbol
@@
     (on_board yes)
     (dnp no)
-    (property "Reference" "C20"
+    (property "Reference" "C19"
       (at 325.12 92.71 90)
       (effects
@@
       (project "electroNIX-USB"
         (path "/af167dc7-e2c9-570c-bdf4-28156a519677/f6fa350a-459e-5361-98c1-1f12d068c3cb"
-          (reference "C20")
+          (reference "C19")
           (unit 1)))))
   (symbol
@@
     (on_board yes)
     (dnp no)
-    (property "Reference" "D4"
+    (property "Reference" "D3"
       (at 186.69 71.12 90)
       (effects
@@
       (project "electroNIX-USB"
         (path "/af167dc7-e2c9-570c-bdf4-28156a519677/f6fa350a-459e-5361-98c1-1f12d068c3cb"
-          (reference "D4")
+          (reference "D3")
           (unit 1)))))
   (symbol
@@
     (on_board yes)
     (dnp no)
-    (property "Reference" "D5"
+    (property "Reference" "D4"
       (at 210.82 71.12 90)
       (effects
@@
       (project "electroNIX-USB"
         (path "/af167dc7-e2c9-570c-bdf4-28156a519677/f6fa350a-459e-5361-98c1-1f12d068c3cb"
-          (reference "D5")
+          (reference "D4")
           (unit 1)))))
   (symbol
@@
     (on_board yes)
     (dnp no)
-    (property "Reference" "D6"
+    (property "Reference" "D5"
       (at 236.22 71.12 90)
       (effects
@@
       (project "electroNIX-USB"
         (path "/af167dc7-e2c9-570c-bdf4-28156a519677/f6fa350a-459e-5361-98c1-1f12d068c3cb"
-          (reference "D6")
+          (reference "D5")
           (unit 1)))))
   (symbol
@@
     (on_board yes)
     (dnp no)
-    (property "Reference" "D7"
+    (property "Reference" "D6"
       (at 261.62 71.12 90)
       (effects
@@
       (project "electroNIX-USB"
         (path "/af167dc7-e2c9-570c-bdf4-28156a519677/f6fa350a-459e-5361-98c1-1f12d068c3cb"
-          (reference "D7")
+          (reference "D6")
           (unit 1)))))
   (symbol
@@
     (on_board yes)
     (dnp no)
-    (property "Reference" "D8"
+    (property "Reference" "D7"
       (at 285.75 71.12 90)
       (effects
@@
       (project "electroNIX-USB"
         (path "/af167dc7-e2c9-570c-bdf4-28156a519677/f6fa350a-459e-5361-98c1-1f12d068c3cb"
-          (reference "D8")
+          (reference "D7")
           (unit 1)))))
   (symbol
@@
     (on_board yes)
     (dnp no)
-    (property "Reference" "D9"
+    (property "Reference" "D8"
       (at 311.15 71.12 90)
       (effects
@@
       (project "electroNIX-USB"
         (path "/af167dc7-e2c9-570c-bdf4-28156a519677/f6fa350a-459e-5361-98c1-1f12d068c3cb"
-          (reference "D9")
+          (reference "D8")
           (unit 1)))))
   (symbol
@@
     (on_board yes)
     (dnp no)
-    (property "Reference" "D10"
+    (property "Reference" "D9"
       (at 336.55 71.12 90)
       (effects
@@
       (project "electroNIX-USB"
         (path "/af167dc7-e2c9-570c-bdf4-28156a519677/f6fa350a-459e-5361-98c1-1f12d068c3cb"
-          (reference "D10")
+          (reference "D9")
           (unit 1)))))
   (symbol
@@
     (on_board yes)
     (dnp no)
-    (property "Reference" "C21"
+    (property "Reference" "C20"
       (at 45.72 163.83 0)
       (effects
@@
       (project "electroNIX-USB"
         (path "/af167dc7-e2c9-570c-bdf4-28156a519677/f6fa350a-459e-5361-98c1-1f12d068c3cb"
-          (reference "C21")
+          (reference "C20")
           (unit 1)))))
   (symbol
@@
     (on_board yes)
     (dnp no)
-    (property "Reference" "R14"
+    (property "Reference" "R11"
       (at 101.6 158.75 0)
       (effects
@@
       (project "electroNIX-USB"
         (path "/af167dc7-e2c9-570c-bdf4-28156a519677/f6fa350a-459e-5361-98c1-1f12d068c3cb"
-          (reference "R14")
+          (reference "R11")
           (unit 1)))))
   (symbol
@@
     (on_board yes)
     (dnp no)
-    (property "Reference" "R15"
+    (property "Reference" "R12"
       (at 101.6 179.07 0)
       (effects
@@
       (project "electroNIX-USB"
         (path "/af167dc7-e2c9-570c-bdf4-28156a519677/f6fa350a-459e-5361-98c1-1f12d068c3cb"
-          (reference "R15")
+          (reference "R12")
           (unit 1)))))
   (symbol
@@
     (on_board yes)
     (dnp no)
-    (property "Reference" "C22"
+    (property "Reference" "C21"
       (at 116.84 173.99 0)
       (effects
@@
       (project "electroNIX-USB"
         (path "/af167dc7-e2c9-570c-bdf4-28156a519677/f6fa350a-459e-5361-98c1-1f12d068c3cb"
-          (reference "C22")
+          (reference "C21")
           (unit 1)))))
   (symbol
@@
     (on_board yes)
     (dnp no)
-    (property "Reference" "D11"
+    (property "Reference" "D10"
       (at 153.67 173.99 0)
       (effects
@@
       (project "electroNIX-USB"
         (path "/af167dc7-e2c9-570c-bdf4-28156a519677/f6fa350a-459e-5361-98c1-1f12d068c3cb"
-          (reference "D11")
+          (reference "D10")
           (unit 1))))))

Commit message: electroNIX-USB: apply RFT Z573M data sheet, add tube footprint
The data book confirms the pinout already in the symbol. The tube is
side-view (not top-view), with 13 flying leads on a 9.53 mm circle and
wire 7 at the front. New footprint electronix:Nixie_RFT_Z573M (top
view, wire 7 toward the front edge) is assigned to the tubes.

Tube current: Ik is 1.5-2.5 mA continuous, 12 mA pulse. PCB-036's 10k
anode resistors averaged only ~0.75 mA per tube when multiplexed. Anode
resistors are now 5k6 (4 tubes) and 3k9 (6 tubes), cathode base
resistors 6k8. To carry the extra HV power, the ladder caps go to
2.2 uF and the 6-tube build uses a 22 uH inductor.

Co-Authored-By: Claude Opus 5.5 <noreply@anthropic.com>
Claude-Session: https://claude.ai/code/session_01AFMfevKEKDGbci8uJGhf4W
Parts:
- C13, C14, C15, C16, C17, C18, C19: value 1u 100V -> 2u2 100V
Other:
- note added: "Cockcroft-Walton multiplier, 7 x 10MQ100N, 7 x 2u2/100V (PCB-036 used 1u)"
- note removed: "Cockcroft-Walton multiplier, 7 x 10MQ100N, 7 x 1u/100V (as PCB-036)"
Changed lines of the file:
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@@
       (type none))
 )
-  (text "Cockcroft-Walton multiplier, 7 x 10MQ100N, 7 x 1u/100V (as PCB-036)"
+  (text "Cockcroft-Walton multiplier, 7 x 10MQ100N, 7 x 2u2/100V (PCB-036 used 1u)"
     (at 161.27 26.27 0)
     (effects
@@
         (font
           (size 1.27 1.27))))
-    (property "Value" "1u 100V"
+    (property "Value" "2u2 100V"
       (at 199.39 52.07 90)
       (effects
@@
         (font
           (size 1.27 1.27))))
-    (property "Value" "1u 100V"
+    (property "Value" "2u2 100V"
       (at 250.19 52.07 90)
       (effects
@@
         (font
           (size 1.27 1.27))))
-    (property "Value" "1u 100V"
+    (property "Value" "2u2 100V"
       (at 299.72 52.07 90)
       (effects
@@
         (font
           (size 1.27 1.27))))
-    (property "Value" "1u 100V"
+    (property "Value" "2u2 100V"
       (at 350.52 52.07 90)
       (effects
@@
         (font
           (size 1.27 1.27))))
-    (property "Value" "1u 100V"
+    (property "Value" "2u2 100V"
       (at 224.79 97.79 90)
       (effects
@@
         (font
           (size 1.27 1.27))))
-    (property "Value" "1u 100V"
+    (property "Value" "2u2 100V"
       (at 275.59 97.79 90)
       (effects
@@
         (font
           (size 1.27 1.27))))
-    (property "Value" "1u 100V"
+    (property "Value" "2u2 100V"
       (at 325.12 97.79 90)
       (effects

Commit message: electroNIX-USB: drop all switches, regroup board placement by circuit
- No RESET/BOOT/SET: the firmware reads no button, and the CH340C
  DTR/RTS auto-reset handles flashing. SET's pull-up and cap are gone.
- Boost converter is a compact loop (input caps -> L1 -> FET tab) feeding
  the multiplier columns in chain order.
- ESP32: 3V3 decoupling at pin 2, EN RC at pin 3, HV feedback divider and
  clamp at IO35; auto-reset between the CH340C and the module's UART pins.
- Front band spread out: output cap + KBIAS left, cathode row, one anode
  cluster under each tube.
- 6-tube board placed too (150 x 66 mm). Both boards unrouted.

Co-Authored-By: Claude Opus 5.5 <noreply@anthropic.com>
Claude-Session: https://claude.ai/code/session_01AFMfevKEKDGbci8uJGhf4W
Parts:
- removed C21: 100n, Capacitor_SMD:C_0805_2012Metric, symbol Device:C
- removed R12: 6k2, Resistor_SMD:R_0805_2012Metric, symbol Device:R
- added C10: 22u 10V, Capacitor_SMD:C_1206_3216Metric, symbol Device:C
- added R8: 10R, Resistor_SMD:R_0805_2012Metric, symbol Device:R
- C11: value 22u 10V -> 100n; footprint Capacitor_SMD:C_1206_3216Metric -> Capacitor_SMD:C_0805_2012Metric
- C12: value 100n -> 2u2 100V; footprint Capacitor_SMD:C_0805_2012Metric -> Capacitor_SMD:C_1210_3225Metric
- C19: value 2u2 100V -> 2u2 250V; footprint Capacitor_SMD:C_1210_3225Metric -> Capacitor_THT:CP_Radial_D6.3mm_P2.50mm; symbol Device:C -> Device:C_Polarized
- C20: value 2u2 250V -> 100n; footprint Capacitor_THT:CP_Radial_D6.3mm_P2.50mm -> Capacitor_SMD:C_0805_2012Metric; symbol Device:C_Polarized -> Device:C
- R10: value 10k -> 430k; footprint Resistor_SMD:R_0805_2012Metric -> Resistor_SMD:R_1206_3216Metric
- R11: value 430k -> 6k2; footprint Resistor_SMD:R_1206_3216Metric -> Resistor_SMD:R_0805_2012Metric
- R9: value 10R -> 10k
Connections:
- net +170V: now also C12.1, C19.1, R10.1; no longer C13.1, C20.1, R11.1
- net +5V: now also C10.1; no longer C12.1
- net CW_B1: now also C17.2, C18.1; no longer C18.2, C19.1
- net CW_B2: now also C16.2, C17.1; no longer C17.2, C18.1
- net CW_B3: now also C16.1; no longer C17.1
- net CW_T1: now also C14.2, C15.1; no longer C15.2, C16.1
- net CW_T2: now also C13.2, C14.1; no longer C14.2, C15.1
- net CW_T3: now also C12.2, C13.1; no longer C13.2, C14.1
- net GND: now also C15.2, C19.2, R11.2, R9.2, C10.2; no longer C12.2, C16.2, R10.2
- net HV_SW: now also C18.2; no longer C19.2
- net KOMP_170V: now also C20.1, R10.2, R11.1; no longer R11.2
- net PWM: now also R8.1; no longer R10.1
- net at Q3.1 (G): now also R8.2; no longer R9.2
Other:
- moved on the sheet: C11, C12, C13, C14, C15, C16, C17, C18, R10, R11, R9
Changed lines of the file:
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@@
     (on_board yes)
     (dnp no)
-    (property "Reference" "C11"
+    (property "Reference" "C10"
       (at 36.83 58.42 0)
       (effects
@@
       (project "electroNIX-USB"
         (path "/af167dc7-e2c9-570c-bdf4-28156a519677/f6fa350a-459e-5361-98c1-1f12d068c3cb"
-          (reference "C11")
+          (reference "C10")
           (unit 1)))))
   (symbol
@@
     (on_board yes)
     (dnp no)
-    (property "Reference" "C12"
+    (property "Reference" "C11"
       (at 48.26 58.42 0)
       (effects
@@
       (project "electroNIX-USB"
         (path "/af167dc7-e2c9-570c-bdf4-28156a519677/f6fa350a-459e-5361-98c1-1f12d068c3cb"
-          (reference "C12")
+          (reference "C11")
           (unit 1)))))
   (symbol
@@
     (on_board yes)
     (dnp no)
-    (property "Reference" "R9"
+    (property "Reference" "R8"
       (at 91.44 77.47 90)
       (effects
@@
       (project "electroNIX-USB"
         (path "/af167dc7-e2c9-570c-bdf4-28156a519677/f6fa350a-459e-5361-98c1-1f12d068c3cb"
-          (reference "R9")
+          (reference "R8")
           (unit 1)))))
   (symbol
@@
     (on_board yes)
     (dnp no)
-    (property "Reference" "R10"
+    (property "Reference" "R9"
       (at 86.36 93.98 0)
       (effects
@@
       (project "electroNIX-USB"
         (path "/af167dc7-e2c9-570c-bdf4-28156a519677/f6fa350a-459e-5361-98c1-1f12d068c3cb"
-          (reference "R10")
+          (reference "R9")
           (unit 1)))))
   (symbol
@@
     (on_board yes)
     (dnp no)
-    (property "Reference" "C13"
+    (property "Reference" "C12"
       (at 199.39 46.99 90)
       (effects
@@
       (project "electroNIX-USB"
         (path "/af167dc7-e2c9-570c-bdf4-28156a519677/f6fa350a-459e-5361-98c1-1f12d068c3cb"
-          (reference "C13")
+          (reference "C12")
           (unit 1)))))
   (symbol
@@
     (on_board yes)
     (dnp no)
-    (property "Reference" "C14"
+    (property "Reference" "C13"
       (at 250.19 46.99 90)
       (effects
@@
       (project "electroNIX-USB"
         (path "/af167dc7-e2c9-570c-bdf4-28156a519677/f6fa350a-459e-5361-98c1-1f12d068c3cb"
-          (reference "C14")
+          (reference "C13")
           (unit 1)))))
   (symbol
@@
     (on_board yes)
     (dnp no)
-    (property "Reference" "C15"
+    (property "Reference" "C14"
       (at 299.72 46.99 90)
       (effects
@@
       (project "electroNIX-USB"
         (path "/af167dc7-e2c9-570c-bdf4-28156a519677/f6fa350a-459e-5361-98c1-1f12d068c3cb"
-          (reference "C15")
+          (reference "C14")
           (unit 1)))))
   (symbol
@@
     (on_board yes)
     (dnp no)
-    (property "Reference" "C16"
+    (property "Reference" "C15"
       (at 350.52 46.99 90)
       (effects
@@
       (project "electroNIX-USB"
         (path "/af167dc7-e2c9-570c-bdf4-28156a519677/f6fa350a-459e-5361-98c1-1f12d068c3cb"
-          (reference "C16")
+          (reference "C15")
           (unit 1)))))
   (symbol
@@
     (on_board yes)
     (dnp no)
-    (property "Reference" "C17"
+    (property "Reference" "C16"
       (at 224.79 92.71 90)
       (effects
@@
       (project "electroNIX-USB"
         (path "/af167dc7-e2c9-570c-bdf4-28156a519677/f6fa350a-459e-5361-98c1-1f12d068c3cb"
-          (reference "C17")
+          (reference "C16")
           (unit 1)))))
   (symbol
@@
     (on_board yes)
     (dnp no)
-    (property "Reference" "C18"
+    (property "Reference" "C17"
       (at 275.59 92.71 90)
       (effects
@@
       (project "electroNIX-USB"
         (path "/af167dc7-e2c9-570c-bdf4-28156a519677/f6fa350a-459e-5361-98c1-1f12d068c3cb"
-          (reference "C18")
+          (reference "C17")
           (unit 1)))))
   (symbol
@@
     (on_board yes)
     (dnp no)
-    (property "Reference" "C19"
+    (property "Reference" "C18"
       (at 325.12 92.71 90)
       (effects
@@
       (project "electroNIX-USB"
         (path "/af167dc7-e2c9-570c-bdf4-28156a519677/f6fa350a-459e-5361-98c1-1f12d068c3cb"
-          (reference "C19")
+          (reference "C18")
           (unit 1)))))
   (symbol
@@
     (on_board yes)
     (dnp no)
-    (property "Reference" "C20"
+    (property "Reference" "C19"
       (at 45.72 163.83 0)
       (effects
@@
       (project "electroNIX-USB"
         (path "/af167dc7-e2c9-570c-bdf4-28156a519677/f6fa350a-459e-5361-98c1-1f12d068c3cb"
-          (reference "C20")
+          (reference "C19")
           (unit 1)))))
   (symbol
@@
     (on_board yes)
     (dnp no)
-    (property "Reference" "R11"
+    (property "Reference" "R10"
       (at 101.6 158.75 0)
       (effects
@@
       (project "electroNIX-USB"
         (path "/af167dc7-e2c9-570c-bdf4-28156a519677/f6fa350a-459e-5361-98c1-1f12d068c3cb"
-          (reference "R11")
+          (reference "R10")
           (unit 1)))))
   (symbol
@@
     (on_board yes)
     (dnp no)
-    (property "Reference" "R12"
+    (property "Reference" "R11"
       (at 101.6 179.07 0)
       (effects
@@
       (project "electroNIX-USB"
         (path "/af167dc7-e2c9-570c-bdf4-28156a519677/f6fa350a-459e-5361-98c1-1f12d068c3cb"
-          (reference "R12")
+          (reference "R11")
           (unit 1)))))
   (symbol
@@
     (on_board yes)
     (dnp no)
-    (property "Reference" "C21"
+    (property "Reference" "C20"
       (at 116.84 173.99 0)
       (effects
@@
       (project "electroNIX-USB"
         (path "/af167dc7-e2c9-570c-bdf4-28156a519677/f6fa350a-459e-5361-98c1-1f12d068c3cb"
-          (reference "C21")
-          (unit 1)))))
-  (symbol
+          (reference "C20")
+          (unit 1)))))
+  (symbol
