File: hardware/electroNIX-USB/kicad-6tube/electroNIX-USB.kicad_pcb (KiCad board)
At the start: 2 copper layers, 150 x 66 mm, 145 parts, among them J1 USB-C (USB 2.0), Q1 MMBT3904, Q10 MMBTA42, Q11 MMBTA92, Q12 MMBTA42, Q13 MMBTA92, Q14 MMBTA42, Q15 MMBTA92, Q16 MMBTA42, Q17 MMBTA42, Q18 MMBTA42, Q19 MMBTA42, Q2 MMBT3904, Q20 MMBTA42, Q21 MMBTA42, Q22 MMBTA42, Q23 MMBTA42, Q24 MMBTA42, Q25 MMBTA42, Q26 MMBTA42, Q27 MMBTA42, Q3 IRLR3110ZPBF, Q4 MMBTA42, Q5 MMBTA92, Q6 MMBTA42, Q7 MMBTA92, Q8 MMBTA42, Q9 MMBTA92, U1 USBLC6-2SC6, U2 AMS1117-3.3, U3 CH340C, U4 ESP32-WROOM-32E-N4

Commit message: electroNIX-USB: clash-free silkscreen, DRC clean-up
- References at 0.8 mm, auto-placed clear of other references, part
  silkscreen, pads and the board edge (inside the part between pads as a
  last resort)
- ESP32: replace the stock 48 mm keep-out zone/courtyard with a body
  courtyard + antenna rule area; module 0.3 mm inside the edge; min drill
  0.2 mm for its exposed-pad vias
- Tube footprints: round pad 1 (the square pad crowded pad 2) with a
  silk pin-1 dot
- KBIAS columns spaced out slightly

DRC on both placed boards: only the stock USB-C footprint's peg-to-pad
clearance remains (plus the expected unrouted nets).

Co-Authored-By: Claude Opus 5.5 <noreply@anthropic.com>
Claude-Session: https://claude.ai/code/session_01AFMfevKEKDGbci8uJGhf4W
Parts:
- moved C1 0.60 mm to (163.5, 105.5)
- moved C22 0.45 mm to (113.8, 149.6)
- moved C24 0.41 mm to (113.8, 153.5)
- moved R53 0.40 mm to (113.8, 145.6)
- moved U4 0.31 mm to (231.5, 116.1)
- moved F1 0.30 mm to (167.1, 105.5)
- moved C21 0.28 mm to (110.2, 149.6)
- moved C23 0.22 mm to (110.2, 153.5)
- moved R52 0.20 mm to (110.2, 145.6)

Commit message: electroNIX-USB: keep every reference beside or inside its own part
Label placement now only accepts spots within ~1 mm of the part and
closer to it than to any other part; otherwise the reference goes inside
the footprint between the pads. Hard cases are retried first. The KBIAS
network moved under the colon, and the auto-reset strip was spaced out
so every label fits at 0.8 mm. DRC: only the stock USB-C footprint item.

Co-Authored-By: Claude Opus 5.5 <noreply@anthropic.com>
Claude-Session: https://claude.ai/code/session_01AFMfevKEKDGbci8uJGhf4W
Parts:
- moved C23 41.1 mm to (150.6, 161.0)
- moved C24 40.7 mm to (153.8, 161.0)
- moved R53 39.8 mm to (152.0, 156.6), turned to 180 degrees
- moved R52 37.5 mm to (146.0, 156.6), turned to 180 degrees
- moved C21 35.9 mm to (144.2, 161.0)
- moved C22 35.5 mm to (147.4, 161.0)
- moved D11 2.50 mm to (116.5, 150.6)
- moved Q16 2.50 mm to (116.5, 146.0)
- moved R36 2.50 mm to (113.4, 146.0)
- moved D12 2.22 mm to (130.4, 150.6)
- moved Q17 2.22 mm to (130.4, 146.0)
- moved R37 2.22 mm to (127.3, 146.0)
- moved R38 1.94 mm to (141.3, 146.0)
- moved D13 1.94 mm to (144.4, 150.6)
- moved Q18 1.94 mm to (144.4, 146.0)
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